Commit message: adding macros for links and joints

File: urdf/krm.xacro (robot description, xacro)
@@ -2,4 +2,5 @@
 <robot xmlns:xacro="http://www.ros.org/wiki/xacro" name="krm">
 <xacro:include filename="$(find krm_description)/urdf/materials.xacro"/>
+<xacro:include filename="$(find krm_description)/urdf/macros.xacro"/>
     <link name="base_link">
         <visual>
@@ -17,4 +18,5 @@
         </collision>
     </link>
+    <xacro:arm_joint name="base_link01"/>
      <link name="link_01">
         <visual>
@@ -32,10 +34,10 @@
         </collision>
     </link>
-    <joint name="base_link01_joint" type="revolute">
-        <origin xyz="0.0 0.0 0.50" rpy="0.0 0.0 0.0"/>
-        <parent link="base_link"/>
-        <child link="link_01"/>
-        <axis xyz="0.0 0.0 1.0"/>
-        <limit lower="-3.14" upper="3.14" effort="1000.0" velocity="0.5"/>
-    </joint>
+    <xacro:arm_link name="02"/>
+    <xacro:arm_joint name="link02_link03"/>
+    <xacro:arm_link name="03"/>
+    <xacro:arm_joint name="link03_link04"/>
+    <xacro:arm_link name="04"/>
+    <xacro:arm_joint name="link04_link05"/>
+    <xacro:arm_link name="05"/>
 </robot>

Commit message: fixing the macro file + increasing robot degree of freedoms

File: urdf/krm.xacro (robot description, xacro)
@@ -3,4 +3,5 @@
 <xacro:include filename="$(find krm_description)/urdf/materials.xacro"/>
 <xacro:include filename="$(find krm_description)/urdf/macros.xacro"/>
+<xacro:include filename="$(find krm_description)/urdf/krm.gazebo"/>
     <link name="base_link">
         <visual>
@@ -18,5 +19,5 @@
         </collision>
     </link>
-    <xacro:arm_joint name="base_link01"/>
+    <xacro:arm_joint name="base_link01"  parent="base_link" child="link_01" axis="0 0 1" />
      <link name="link_01">
         <visual>
@@ -34,10 +35,11 @@
         </collision>
     </link>
-    <xacro:arm_link name="02"/>
-    <xacro:arm_joint name="link02_link03"/>
-    <xacro:arm_link name="03"/>
-    <xacro:arm_joint name="link03_link04"/>
-    <xacro:arm_link name="04"/>
-    <xacro:arm_joint name="link04_link05"/>
-    <xacro:arm_link name="05"/>
+    <xacro:arm_joint name="link01_link02" parent="link_01" child="link_02" axis="1 0 0" />
+    <xacro:arm_link name="link_02"/>
+    <xacro:arm_joint name="link02_link03" parent="link_02" child="link_03" axis="1 0 0"/>
+    <xacro:arm_link name="link_03"/>
+    <xacro:arm_joint name="link03_link04" parent="link_03" child="link_04" axis="1 0 0"/>
+    <xacro:arm_link name="link_04"/>
+    <xacro:arm_joint name="link04_link05" parent="link_04" child="link_05" axis="1 0 0"/>
+    <xacro:arm_link name="link_05"/>
 </robot>

File: urdf/macros.xacro (robot description, xacro)
@@ -2,7 +2,7 @@
 <robot>
     <macro name="arm_link" params="name">
-        <link name="link_${name}">
+        <link name="${name}">
             <visual>
-                <origin xyz="0.0 0.0 0.4" rpy="0.0 0.0 0.0"/>
+                <origin xyz="0.0 0.0 0.1" rpy="0.0 0.0 0.0"/>
                 <geometry>
                     <cylinder radius="0.15" length="0.8"/>
@@ -18,10 +18,10 @@
         </link>
     </macro>
-    <macro name="arm_joint" params="name parent child ">
+    <macro name="arm_joint" params="name parent child axis">
         <joint name="${name}_joint" type="revolute">
-            <origin xyz="0.0 0.0 0.50" rpy="0.0 0.0 0.0"/>
+            <origin xyz="0.0 0.0 0.7" rpy="0.0 0.0 0.0"/>
             <parent link="${parent}"/>
             <child link="${child}"/>
-            <axis xyz="0.0 0.0 1.0"/>
+            <axis xyz="${axis}"/>
             <limit lower="-3.14" upper="3.14" effort="1000.0" velocity="0.5"/>
         </joint>

Commit message: inertia and mass for links

File: urdf/krm.xacro (robot description, xacro)
@@ -35,11 +35,27 @@
         </collision>
     </link>
-    <xacro:arm_joint name="link01_link02" parent="link_01" child="link_02" axis="1 0 0" />
+    <xacro:arm_joint name="link01_link02"
+    parent="link_01"
+    child="link_02"
+    axis="1 0 0"
+    />
     <xacro:arm_link name="link_02"/>
-    <xacro:arm_joint name="link02_link03" parent="link_02" child="link_03" axis="1 0 0"/>
+    <xacro:arm_joint name="link02_link03"
+    parent="link_02"
+    child="link_03"
+    axis="1 0 0"
+    />
     <xacro:arm_link name="link_03"/>
-    <xacro:arm_joint name="link03_link04" parent="link_03" child="link_04" axis="1 0 0"/>
+    <xacro:arm_joint name="link03_link04"
+    parent="link_03"
+    child="link_04"
+    axis="1 0 0"
+    />
     <xacro:arm_link name="link_04"/>
-    <xacro:arm_joint name="link04_link05" parent="link_04" child="link_05" axis="1 0 0"/>
+    <xacro:arm_joint name="link04_link05"
+    parent="link_04"
+    child="link_05"
+    axis="1 0 0"
+    />
     <xacro:arm_link name="link_05"/>
 </robot>

File: urdf/macros.xacro (robot description, xacro)
@@ -3,4 +3,9 @@
     <macro name="arm_link" params="name">
         <link name="${name}">
+            <inertial>
+                <origin xyz="0.0 0.0 0.0" rpy="0.0 0.0 0.4"/>
+                <mass value="57.904"/>
+                <inertia ixx="12.679" ixy="0.0" ixz="0.0" iyy="12.679" iyz="0.0" izz="0.651"/>
+            </inertial>
             <visual>
                 <origin xyz="0.0 0.0 0.1" rpy="0.0 0.0 0.0"/>

Commit message: ros

File: urdf/krm.xacro (robot description, xacro)
@@ -19,5 +19,9 @@
         </collision>
     </link>
-    <xacro:arm_joint name="base_link01"  parent="base_link" child="link_01" axis="0 0 1" />
+    <xacro:arm_joint name="base_link01"
+    parent="base_link"
+    child="link_01"
+    axis="0 0 1" />
+    <xacro:joint_trans name="base_link01"/>
      <link name="link_01">
         <visual>
@@ -40,6 +44,7 @@
     axis="1 0 0"
     />
+     <xacro:joint_trans name="link01_link02"/>
     <xacro:arm_link name="link_02"/>
-    <xacro:arm_joint name="link02_link03"
+    <!--xacro:arm_joint name="link02_link03"
     parent="link_02"
     child="link_03"
@@ -58,4 +63,4 @@
     axis="1 0 0"
     />
-    <xacro:arm_link name="link_05"/>
+    <xacro:arm_link name="link_05"/-->
 </robot>

File: urdf/macros.xacro (robot description, xacro)
@@ -16,5 +16,5 @@
             </visual>
             <collision>
-                <origin xyz="0.0 0.0 0.4" rpy="0.0 0.0 0.0"/>
+                <origin xyz="0.0 0.0 0.1" rpy="0.0 0.0 0.0"/>
                 <geometry>
                     <cylinder radius="0.15" length="0.8"/>
@@ -25,5 +25,5 @@
     <macro name="arm_joint" params="name parent child axis">
         <joint name="${name}_joint" type="revolute">
-            <origin xyz="0.0 0.0 0.7" rpy="0.0 0.0 0.0"/>
+            <origin xyz="0.0 0.0 0.6" rpy="0.0 0.0 0.0"/>
             <parent link="${parent}"/>
             <child link="${child}"/>
@@ -32,3 +32,15 @@
         </joint>
     </macro>
+    <macro name="joint_trans" params="name ">
+        <transmission name="${name}_trans">
+            <type>transmission_interface/SimpleTransmission</type>
+            <joint name="${name}">
+                <hardwareInterface>EffortJointInterface</hardwareInterface>
+            </joint>
+            <actuator name="${name}_motor">
+                <mechanicalReduction>1</mechanicalReduction>
+                <hardwareInterface>EffortJointInterface</hardwareInterface>
+            </actuator>
+        </transmission>
+    </macro>
 </robot>
